Commit message: milestone: fix bugs and make a successful training

File: resources/environment/wall.urdf (robot description, URDF)
Before this commit: robot arena, 1 links, 0 joints
Links:
- removed link arena_base
- added link wall, mass 0.001; collision box size=1 0.05 0.5; visual box size=1 0.05 0.5
